File: SMPS Breakout Board.kicad_pcb (KiCad board)
At the start: 2 copper layers, 60 x 40 mm, 27 parts, among them J1 Screw_Terminal_01x02, J2 Conn_01x02_Male, J3 Screw_Terminal_01x02, J4 Conn_01x03_Male, J6 Conn_01x02_Male, U1 LM2596S-3.3, U2 INA169

Commit message: More finishing touches, all parts have an LCSC number
Parts:
- C1: footprint Capacitor_SMD:CP_Elec_10x10.5 -> Capacitor_SMD:CP_Elec_10x12.5
- D1: value 1N5824 -> 1N5821
- J1, J3: footprint TerminalBlock:TerminalBlock_bornier-2_P5.08mm -> TerminalBlock_Phoenix:TerminalBlock_Phoenix_MKDS-1,5-2_1x02_P5.00mm_Horizontal
- L1: value L -> 22uH
- R1: value R -> 0.1 2W; footprint Resistor_SMD:R_2816_7142Metric -> Resistor_SMD:R_2512_6332Metric
- R2: value R -> 10K
- moved R3 3.18 mm to (146.1, 146.5), turned to 0 degrees
- moved R4 1.34 mm to (146.1, 149.0), turned to 180 degrees
- moved J4 0.85 mm to (144.5, 153.7)
- moved R1 0.84 mm to (145.6, 142.6)
- moved J6 0.67 mm to (155.7, 137.4)
- moved C4 0.56 mm to (138.8, 134.0)
- moved J1 0.48 mm to (105.5, 143.0)
- moved C1 0.47 mm to (109.7, 134.3)
- moved C7 0.16 mm to (150.0, 137.6)
- moved L1 0.12 mm to (134.9, 147.4)
Routing:
- net VOLT_SENSE: track 5.99 -> 7.92 mm
- net Net-(J3-Pad2): track 26.2 -> 26.9 mm
- net Net-(D1-Pad1): track 15.9 -> 15.2 mm
- net CURRENT_SENSE: track 23.6 -> 24.3 mm
- net GND: vias 151 -> 150
Other:
- board text added: "+ -"
- board text added: "- V C"
- board text added: "VIn"
- board text added: "VOut"
